File: XenoGCFlex.kicad_pcb (KiCad board)
At the start: 2 copper layers, 23.6 x 20 mm, 21 parts, among them J1 AVR-ISP-6, U1 ATmega8A-AU

Commit message: Remove text
Other:
- board text removed: "Put this side towards the board Or don't i'm a PCB not a cop."
Changed lines of the file:
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@@
   (general
     (thickness 1.6)
-    (drawings 18)
+    (drawings 17)
     (tracks 146)
     (zones 0)
@@
     )
   )
-  (gr_text "Put this side towards the board\nOr don't i'm a PCB not a cop." (at 145.33118 79.16222) (layer B.SilkS)
-    (effects (font (size 0.5 0.5) (thickness 0.1)) (justify mirror))
-  )
   (gr_text MartinRefseth.com (at 149.291 72.407 315) (layer F.SilkS)
